Commit message: 初步实现整个架构重写以及调试

File: ros2_master/src/amr/amr_launch/urdf/amr_real.xacro (robot description, xacro)
@@ -2,7 +2,7 @@
 <robot xmlns:xacro="http://ros.org/wiki/xacro" name="amr_real">
     <xacro:property name="base_link" value="base_link" />
-    <xacro:property name="lidar_link" value="lidar_frame" />
-    <xacro:property name="camera_link" value="camera_frame" />
-    <xacro:property name="imu_link" value="imu_frame" />
+    <xacro:property name="lidar_link" value="lidar_link" />
+    <xacro:property name="camera_link" value="camera_link" />
+    <xacro:property name="imu_link" value="imu_link" />
     <xacro:property name="left_front_wheel" value="left_front_wheel" />
     <xacro:property name="left_back_wheel" value="left_back_wheel" />

File: ros2_master/src/amr/amr_launch/urdf/amr_sim.xacro (robot description, xacro)
@@ -2,7 +2,7 @@
 <robot xmlns:xacro="http://ros.org/wiki/xacro" name="amr_sim">
     <xacro:property name="base_link" value="base_link" />
-    <xacro:property name="lidar_link" value="lidar_frame" />
-    <xacro:property name="camera_link" value="camera_frame" />
-    <xacro:property name="imu_link" value="imu_frame" />
+    <xacro:property name="lidar_link" value="lidar_link" />
+    <xacro:property name="camera_link" value="camera_link" />
+    <xacro:property name="imu_link" value="imu_link" />
     <xacro:property name="left_wheel" value="left_wheel" />
     <xacro:property name="right_wheel" value="right_wheel" />
