Commit message: 修复bug

File: ros2_master/src/description/urdf/amr_description.xacro (robot description, xacro)
@@ -13,10 +13,10 @@
     <xacro:property name="front_castor" value="front_castor" />
     <xacro:property name="back_castor" value="back_castor" />
-    <xacro:include filename="$(find amr_launch)/urdf/base.xacro" />
-    <xacro:include filename="$(find amr_launch)/urdf/wheel.xacro" />
-    <xacro:include filename="$(find amr_launch)/urdf/castor.xacro" />
-    <xacro:include filename="$(find amr_launch)/urdf/lidar.xacro" />
-    <xacro:include filename="$(find amr_launch)/urdf/camera.xacro" />
-    <xacro:include filename="$(find amr_launch)/urdf/imu.xacro" />
+    <xacro:include filename="$(find description)/urdf/base.xacro" />
+    <xacro:include filename="$(find description)/urdf/wheel.xacro" />
+    <xacro:include filename="$(find description)/urdf/castor.xacro" />
+    <xacro:include filename="$(find description)/urdf/lidar.xacro" />
+    <xacro:include filename="$(find description)/urdf/camera.xacro" />
+    <xacro:include filename="$(find description)/urdf/imu.xacro" />
     <xacro:base name="${base_link}" joint_xyz="0 0 ${wheel_radius}" />
     <xacro:lidar name="${lidar_link}" joint_xyz="-${base_width/4} 0 ${lidar_height/2}" parent_name="${base_link}" />

File: ros2_master/src/description/urdf/amr_real.xacro (robot description, xacro)
@@ -9,9 +9,9 @@
     <xacro:property name="right_front_wheel" value="right_front_wheel" />
     <xacro:property name="right_back_wheel" value="right_back_wheel" />
-    <xacro:include filename="$(find amr_launch)/urdf/base.xacro" />
-    <xacro:include filename="$(find amr_launch)/urdf/wheel.xacro" />
-    <xacro:include filename="$(find amr_launch)/urdf/lidar.xacro" />
-    <xacro:include filename="$(find amr_launch)/urdf/camera.xacro" />
-    <xacro:include filename="$(find amr_launch)/urdf/imu.xacro" />
+    <xacro:include filename="$(find description)/urdf/base.xacro" />
+    <xacro:include filename="$(find description)/urdf/wheel.xacro" />
+    <xacro:include filename="$(find description)/urdf/lidar.xacro" />
+    <xacro:include filename="$(find description)/urdf/camera.xacro" />
+    <xacro:include filename="$(find description)/urdf/imu.xacro" />
     <xacro:base name="${base_link}" joint_xyz="0 0 ${wheel_radius}" />
     <xacro:lidar name="${lidar_link}" joint_xyz="-${base_width/4} 0 ${lidar_height/2}" parent_name="${base_link}" />

File: ros2_master/src/description/urdf/amr_sim.xacro (robot description, xacro)
@@ -9,10 +9,10 @@
     <xacro:property name="front_castor" value="front_castor" />
     <xacro:property name="back_castor" value="back_castor" />
-    <xacro:include filename="$(find amr_launch)/urdf/base.xacro" />
-    <xacro:include filename="$(find amr_launch)/urdf/wheel.xacro" />
-    <xacro:include filename="$(find amr_launch)/urdf/castor.xacro" />
-    <xacro:include filename="$(find amr_launch)/urdf/lidar.xacro" />
-    <xacro:include filename="$(find amr_launch)/urdf/camera.xacro" />
-    <xacro:include filename="$(find amr_launch)/urdf/imu.xacro" />
+    <xacro:include filename="$(find description)/urdf/base.xacro" />
+    <xacro:include filename="$(find description)/urdf/wheel.xacro" />
+    <xacro:include filename="$(find description)/urdf/castor.xacro" />
+    <xacro:include filename="$(find description)/urdf/lidar.xacro" />
+    <xacro:include filename="$(find description)/urdf/camera.xacro" />
+    <xacro:include filename="$(find description)/urdf/imu.xacro" />
     <xacro:base name="${base_link}" joint_xyz="0 0 ${wheel_radius}" />
     <xacro:lidar name="${lidar_link}" joint_xyz="-${base_width/4} 0 ${lidar_height/2}" parent_name="${base_link}" />
@@ -23,5 +23,5 @@
     <xacro:castor name="${front_castor}" joint_xyz="${base_length/2-castor_radius} 0 -${castor_radius}" parent_name="${base_link}" />
     <xacro:castor name="${back_castor}" joint_xyz="-${base_length/2-castor_radius} 0 -${castor_radius}" parent_name="${base_link}" />
-    <xacro:include filename="$(find amr_launch)/urdf/gazebo_sensors_plugins.xacro" />
+    <xacro:include filename="$(find description)/urdf/gazebo_sensors_plugins.xacro" />
     <xacro:gazebo_sensors_plugins camera_link="${camera_link}" lidar_link="${lidar_link}" imu_link="${imu_link}" />
     <ros2_control name="ros2_controllers" type="system">
@@ -42,5 +42,5 @@
     <gazebo>
         <plugin filename="libgz_ros2_control-system.so" name="gz_ros2_control::GazeboSimROS2ControlPlugin">
-            <parameters>$(find amr_launch)/config/ros2_controllers_sim.yaml</parameters>
+            <parameters>$(find description)/config/ros2_controllers_sim.yaml</parameters>
         </plugin>
     </gazebo>

File: ros2_master/src/description/urdf/base.xacro (robot description, xacro)
@@ -1,5 +1,5 @@
 <?xml version="1.0"?>
 <robot xmlns:xacro="http://ros.org/wiki/xacro" name="base">
-    <xacro:include filename="$(find amr_launch)/urdf/common_inertia.xacro" />
+    <xacro:include filename="$(find description)/urdf/common_inertia.xacro" />
     <xacro:property name="base_length" value="0.120" />
     <xacro:property name="base_width" value="0.080" />

File: ros2_master/src/description/urdf/camera.xacro (robot description, xacro)
@@ -1,5 +1,5 @@
 <?xml version="1.0"?>
 <robot xmlns:xacro="http://ros.org/wiki/xacro">
-    <xacro:include filename="$(find amr_launch)/urdf/common_inertia.xacro" />
+    <xacro:include filename="$(find description)/urdf/common_inertia.xacro" />
     <xacro:property name="camera_length" value="0.025" />
     <xacro:property name="camera_width" value="0.01" />

File: ros2_master/src/description/urdf/castor.xacro (robot description, xacro)
@@ -1,5 +1,5 @@
 <?xml version="1.0"?>
 <robot xmlns:xacro="http://ros.org/wiki/xacro">
-    <xacro:include filename="$(find amr_launch)/urdf/common_inertia.xacro" />
+    <xacro:include filename="$(find description)/urdf/common_inertia.xacro" />
     <xacro:property name="castor_radius" value="0.020" />
     <xacro:property name="wheel_mass" value="0.01" />

File: ros2_master/src/description/urdf/imu.xacro (robot description, xacro)
@@ -1,4 +1,4 @@
 <robot xmlns:xacro="http://ros.org/wiki/xacro">
-    <xacro:include filename="$(find amr_launch)/urdf/common_inertia.xacro" />
+    <xacro:include filename="$(find description)/urdf/common_inertia.xacro" />
     <xacro:property name="imu_length" value="0.01" />
     <xacro:property name="imu_width" value="0.02" />

File: ros2_master/src/description/urdf/lidar.xacro (robot description, xacro)
@@ -1,5 +1,5 @@
 <?xml version="1.0"?>
 <robot xmlns:xacro="http://ros.org/wiki/xacro">
-    <xacro:include filename="$(find amr_launch)/urdf/common_inertia.xacro" />
+    <xacro:include filename="$(find description)/urdf/common_inertia.xacro" />
     <xacro:property name="lidar_radius" value="0.015" />
     <xacro:property name="lidar_height" value="0.060" />

File: ros2_master/src/description/urdf/ros2_controllers.xacro (robot description, xacro)
@@ -47,5 +47,5 @@
     <gazebo>
         <plugin filename="libgz_ros2_control-system.so" name="gz_ros2_control::GazeboSimROS2ControlPlugin">
-            <parameters>$(find amr_launch)/config/ros2_controllers.yaml</parameters>
+            <parameters>$(find description)/config/ros2_controllers.yaml</parameters>
         </plugin>
     </gazebo>

File: ros2_master/src/description/urdf/wheel.xacro (robot description, xacro)
@@ -1,5 +1,5 @@
 <?xml version="1.0"?>
 <robot xmlns:xacro="http://ros.org/wiki/xacro">
-    <xacro:include filename="$(find amr_launch)/urdf/common_inertia.xacro" />
+    <xacro:include filename="$(find description)/urdf/common_inertia.xacro" />
     <xacro:property name="wheel_radius" value="0.040" />
     <xacro:property name="wheel_width" value="0.040" />
@@ -13,5 +13,5 @@
                 <geometry>
                     <cylinder radius="${wheel_radius}" length="${wheel_width}" />
-                    <!-- <mesh filename="file://$(find amr_launch)/mesh/wheel/${name}.dae" /> -->
+                    <!-- <mesh filename="file://$(find description)/mesh/wheel/${name}.dae" /> -->
                 </geometry>
                 <material name="yellow">
