Commit message: 修复调试出现的bug

File: ros2_master/src/description/urdf/base.xacro (robot description, xacro)
@@ -1,9 +1,7 @@
 <?xml version="1.0"?>
 <robot xmlns:xacro="http://ros.org/wiki/xacro" name="base">
-    <xacro:include filename="$(find description)/urdf/common_inertia.xacro" />
-    <xacro:property name="base_length" value="0.120" />
-    <xacro:property name="base_width" value="0.080" />
-    <xacro:property name="base_height" value="0.006" />
-    <xacro:property name="base_mass" value="1.0" />
+    <xacro:property name="base_length" value="0.210" />
+    <xacro:property name="base_width" value="0.120" />
+    <xacro:property name="base_height" value="0.009" />
     <xacro:property name="link_xyz" value="0 0 0" />
     <xacro:property name="link_rpy" value="0 0 0" />
@@ -26,5 +24,4 @@
                 </geometry>
             </collision>
-            <xacro:box_inertia m="${base_mass}" w="${base_length}" h="${base_height}" d="${base_width}" xyz="${link_xyz}" rpy="${link_rpy}" />
         </link>
         <joint name="${name}_joint" type="fixed">

File: ros2_master/src/description/urdf/camera.xacro (robot description, xacro)
@@ -1,13 +1,7 @@
 <?xml version="1.0"?>
 <robot xmlns:xacro="http://ros.org/wiki/xacro">
-    <xacro:include filename="$(find description)/urdf/common_inertia.xacro" />
-    <xacro:property name="camera_length" value="0.025" />
-    <xacro:property name="camera_width" value="0.01" />
-    <xacro:property name="camera_height" value="0.01" />
-    <xacro:property name="camera_mass" value="0.1" />
-    <xacro:property name="camera_support_length" value="0.005" />
-    <xacro:property name="camera_support_width" value="0.005" />
-    <xacro:property name="camera_support_height" value="0.04" />
-    <xacro:property name="camera_support_mass" value="0.01" />
+    <xacro:property name="camera_length" value="0.019" />
+    <xacro:property name="camera_width" value="0.027" />
+    <xacro:property name="camera_height" value="0.042" />
     <xacro:macro name="camera" params="name joint_xyz parent_name">
         <link name="${name}">
@@ -27,34 +21,9 @@
                 </geometry>
             </collision>
-            <xacro:box_inertia m="${camera_mass}" w="${camera_width}" h="${camera_length}" d="${camera_height}" xyz="0 0 0" rpy="0 0 0" />
         </link>
-        <xacro:property name="support_name" value="support_${name}" />
-        <link name="${support_name}">
-            <visual>
-                <origin xyz="0 0 0" rpy="0 0 0" />
-                <geometry>
-                    <box size="${camera_support_width} ${camera_support_length} ${camera_support_height}" />
-                </geometry>
-                <material name="grey">
-                    <color rgba="0.5 0.5 0.5 1" />
-                </material>
-            </visual>
-            <collision>
-                <origin xyz="0 0 0" rpy="0 0 0" />
-                <geometry>
-                    <box size="${camera_support_width} ${camera_support_length} ${camera_support_height}" />
-                </geometry>
-            </collision>
-            <xacro:box_inertia m="${camera_support_mass}" w="${camera_support_width}" h="${camera_support_length}" d="${camera_support_height}" xyz="0 0 0" rpy="0 0 0" />
-        </link>
-        <joint name="${support_name}_joint" type="fixed">
+        <joint name="${name}_joint" type="fixed">
             <parent link="${parent_name}" />
-            <child link="${support_name}" />
+            <child link="${name}" />
             <origin xyz="${joint_xyz}" rpy="0 0 0" />
-        </joint>
-        <joint name="${name}_joint" type="fixed">
-            <parent link="${support_name}" />
-            <child link="${name}" />
-            <origin xyz="0 0 ${camera_support_height/2}" rpy="0 0 0" />
         </joint>
     </xacro:macro>

File: ros2_master/src/description/urdf/imu.xacro (robot description, xacro)
@@ -1,8 +1,6 @@
 <robot xmlns:xacro="http://ros.org/wiki/xacro">
-    <xacro:include filename="$(find description)/urdf/common_inertia.xacro" />
-    <xacro:property name="imu_length" value="0.01" />
-    <xacro:property name="imu_width" value="0.02" />
-    <xacro:property name="imu_height" value="0.003" />
-    <xacro:property name="imu_mass" value="0.005" />
+    <xacro:property name="imu_length" value="0.016" />
+    <xacro:property name="imu_width" value="0.021" />
+    <xacro:property name="imu_height" value="0.0015" />
     <xacro:macro name="imu" params="name joint_xyz parent_name">
         <link name="${name}">
@@ -22,5 +20,4 @@
                 </geometry>
             </collision>
-            <xacro:box_inertia m="${imu_mass}" w="${imu_length}" h="${imu_width}" d="${imu_height}" xyz="0 0 0" rpy="0 0 0" />
         </link>
         <joint name="${name}_joint" type="fixed">

File: ros2_master/src/description/urdf/lidar.xacro (robot description, xacro)
@@ -1,12 +1,6 @@
 <?xml version="1.0"?>
 <robot xmlns:xacro="http://ros.org/wiki/xacro">
-    <xacro:include filename="$(find description)/urdf/common_inertia.xacro" />
-    <xacro:property name="lidar_radius" value="0.015" />
-    <xacro:property name="lidar_height" value="0.060" />
-    <xacro:property name="lidar_mass" value="0.1" />
-    <xacro:property name="lidar_length" value="${lidar_radius/2}" />
-    <xacro:property name="lidar_support_radius" value="${lidar_radius/4}" />
-    <xacro:property name="lidar_support_length" value="${lidar_height}" />
-    <xacro:property name="lidar_support_mass" value="0.01" />
+    <xacro:property name="lidar_radius" value="0.0325" />
+    <xacro:property name="lidar_height" value="0.020" />
     <xacro:macro name="lidar" params="name joint_xyz parent_name">
         <link name="${name}">
@@ -14,7 +8,6 @@
                 <origin xyz="0 0 0" rpy="0 0 0" />
                 <geometry>
-                    <cylinder radius="${lidar_radius}" length="${lidar_length}" />
-                </geometry>
-                <material name="black">
+                    <cylinder radius="${lidar_radius}" length="${lidar_height}" />
+                </geometry>· <material name="black">
                     <color rgba="0.0 0.0 1.0 1" />
                 </material>
@@ -23,37 +16,12 @@
                 <origin xyz="0 0 0" rpy="0 0 0" />
                 <geometry>
-                    <cylinder radius="${lidar_radius}" length="${lidar_length}" />
+                    <cylinder radius="${lidar_radius}" length="${lidar_height}" />
                 </geometry>
             </collision>
-            <xacro:cylinder_inertia m="${lidar_mass}" r="${lidar_radius}" h="${lidar_length}" xyz="0 0 0" rpy="0 0 0" />
         </link>
-        <xacro:property name="support_name" value="support_${name}" />
-        <link name="${support_name}">
-            <visual>
-                <origin xyz="0 0 0" rpy="0 0 0" />
-                <geometry>
-                    <cylinder radius="${lidar_support_radius}" length="${lidar_support_length}" />
-                </geometry>
-                <material name="grey">
-                    <color rgba="0.5 0.5 0.5 1" />
-                </material>
-            </visual>
-            <collision>
-                <origin xyz="0 0 0" rpy="0 0 0" />
-                <geometry>
-                    <cylinder radius="${lidar_support_radius}" length="${lidar_support_length}" />
-                </geometry>
-            </collision>
-            <xacro:cylinder_inertia m="${lidar_support_mass}" r="${lidar_support_radius}" h="${lidar_support_length}" xyz="0 0 0" rpy="0 0 0" />
-        </link>
-        <joint name="${support_name}_joint" type="fixed">
+        <joint name="${name}_joint" type="fixed">
             <parent link="${parent_name}" />
-            <child link="${support_name}" />
+            <child link="${name}" />
             <origin xyz="${joint_xyz}" rpy="0 0 0" />
-        </joint>
-        <joint name="${name}_joint" type="fixed">
-            <parent link="${support_name}" />
-            <child link="${name}" />
-            <origin xyz="0 0 ${lidar_height/2}" rpy="0 0 0" />
         </joint>
     </xacro:macro>

File: ros2_master/src/description/urdf/wheel.xacro (robot description, xacro)
@@ -1,11 +1,9 @@
 <?xml version="1.0"?>
 <robot xmlns:xacro="http://ros.org/wiki/xacro">
-    <xacro:include filename="$(find description)/urdf/common_inertia.xacro" />
-    <xacro:property name="wheel_radius" value="0.040" />
-    <xacro:property name="wheel_width" value="0.040" />
-    <xacro:property name="wheel_mass" value="0.5" />
+    <xacro:property name="wheel_radius" value="0.0325" />
+    <xacro:property name="wheel_width" value="0.026" />
     <xacro:property name="link_xyz" value="0 0 0" />
     <xacro:property name="link_rpy" value="${pi/2} 0 0" />
-    <xacro:macro name="wheel" params="name joint_xyz fdir1_value parent_name">
+    <xacro:macro name="wheel" params="name joint_xyz parent_name">
         <link name='${name}'>
             <visual>
@@ -13,5 +11,4 @@
                 <geometry>
                     <cylinder radius="${wheel_radius}" length="${wheel_width}" />
-                    <!-- <mesh filename="file://$(find description)/mesh/wheel/${name}.dae" /> -->
                 </geometry>
                 <material name="yellow">
@@ -25,12 +22,5 @@
                 </geometry>
             </collision>
-            <xacro:cylinder_inertia m="${wheel_mass}" r="${wheel_radius}" h="${wheel_width}" xyz="${link_xyz}" rpy="${link_rpy}" />
         </link>
-        <gazebo reference="${name}">
-            <mu1>20.0</mu1>
-            <mu2>20.0</mu2>
-            <kp>10000000</kp>
-            <kd>1.0</kd>
-        </gazebo>
         <joint name="${name}_joint" type="continuous">
             <parent link="${parent_name}" />

File: ros2_master/src/simulation/urdf/amr.xacro (robot description, xacro)
@@ -1,4 +1,4 @@
 <?xml version="1.0"?>
-<robot xmlns:xacro="http://ros.org/wiki/xacro" name="amr_sim">
+<robot xmlns:xacro="http://ros.org/wiki/xacro" name="amr">
     <xacro:property name="base_link" value="base_link" />
     <xacro:property name="lidar_link" value="lidar_link" />
@@ -9,10 +9,10 @@
     <xacro:property name="front_castor" value="front_castor" />
     <xacro:property name="back_castor" value="back_castor" />
-    <xacro:include filename="$(find description)/urdf/base.xacro" />
-    <xacro:include filename="$(find description)/urdf/wheel.xacro" />
-    <xacro:include filename="$(find description)/urdf/castor.xacro" />
-    <xacro:include filename="$(find description)/urdf/lidar.xacro" />
-    <xacro:include filename="$(find description)/urdf/camera.xacro" />
-    <xacro:include filename="$(find description)/urdf/imu.xacro" />
+    <xacro:include filename="$(find simulation)/urdf/base.xacro" />
+    <xacro:include filename="$(find simulation)/urdf/wheel.xacro" />
+    <xacro:include filename="$(find simulation)/urdf/castor.xacro" />
+    <xacro:include filename="$(find simulation)/urdf/lidar.xacro" />
+    <xacro:include filename="$(find simulation)/urdf/camera.xacro" />
+    <xacro:include filename="$(find simulation)/urdf/imu.xacro" />
     <xacro:base name="${base_link}" joint_xyz="0 0 ${wheel_radius}" />
     <xacro:lidar name="${lidar_link}" joint_xyz="-${base_width/4} 0 ${lidar_height/2}" parent_name="${base_link}" />
@@ -23,5 +23,5 @@
     <xacro:castor name="${front_castor}" joint_xyz="${base_length/2-castor_radius} 0 -${castor_radius}" parent_name="${base_link}" />
     <xacro:castor name="${back_castor}" joint_xyz="-${base_length/2-castor_radius} 0 -${castor_radius}" parent_name="${base_link}" />
-    <xacro:include filename="$(find description)/urdf/gazebo_sensors_plugins.xacro" />
+    <xacro:include filename="$(find simulation)/urdf/gazebo_sensors_plugins.xacro" />
     <xacro:gazebo_sensors_plugins camera_link="${camera_link}" lidar_link="${lidar_link}" imu_link="${imu_link}" />
     <ros2_control name="ros2_controllers" type="system">
@@ -42,5 +42,5 @@
     <gazebo>
         <plugin filename="libgz_ros2_control-system.so" name="gz_ros2_control::GazeboSimROS2ControlPlugin">
-            <parameters>$(find description)/config/ros2_controllers_sim.yaml</parameters>
+            <parameters>$(find simulation)/config/ros2_controllers.yaml</parameters>
         </plugin>
     </gazebo>

File: ros2_master/src/simulation/urdf/castor.xacro (robot description, xacro)
@@ -1,5 +1,5 @@
 <?xml version="1.0"?>
 <robot xmlns:xacro="http://ros.org/wiki/xacro">
-    <xacro:include filename="$(find description)/urdf/common_inertia.xacro" />
+    <xacro:include filename="$(find simulation)/urdf/common_inertia.xacro" />
     <xacro:property name="castor_radius" value="0.020" />
     <xacro:property name="wheel_mass" value="0.01" />

File: ros2_master/src/simulation/urdf/ros2_controllers.xacro (robot description, xacro)
@@ -47,5 +47,5 @@
     <gazebo>
         <plugin filename="libgz_ros2_control-system.so" name="gz_ros2_control::GazeboSimROS2ControlPlugin">
-            <parameters>$(find description)/config/ros2_controllers.yaml</parameters>
+            <parameters>$(find simulation)/config/ros2_controllers.yaml</parameters>
         </plugin>
     </gazebo>
