Commit message: 调试各个模块

File: ros2_master/src/description/urdf/amr.xacro (robot description, xacro)
@@ -1,12 +1,14 @@
 <?xml version="1.0"?>
 <robot xmlns:xacro="http://ros.org/wiki/xacro" name="amr">
+    <xacro:property name="track_width" value="0.110" />
+    <xacro:property name="wheel_width" value="0.168" />
     <xacro:property name="base_link" value="base_link" />
     <xacro:property name="lidar_link" value="lidar_link" />
     <xacro:property name="camera_link" value="camera_link" />
     <xacro:property name="imu_link" value="imu_link" />
-    <xacro:property name="left_front_wheel" value="left_front_wheel" />
-    <xacro:property name="left_back_wheel" value="left_back_wheel" />
-    <xacro:property name="right_front_wheel" value="right_front_wheel" />
-    <xacro:property name="right_back_wheel" value="right_back_wheel" />
+    <xacro:property name="chassis_link" value="chassis_link" />
+    <xacro:property name="castor_link" value="castor_link" />
+    <xacro:property name="left_wheel" value="left_wheel" />
+    <xacro:property name="right_wheel" value="right_wheel" />
     <xacro:include filename="$(find description)/urdf/base.xacro" />
     <xacro:include filename="$(find description)/urdf/wheel.xacro" />
@@ -14,11 +16,14 @@
     <xacro:include filename="$(find description)/urdf/camera.xacro" />
     <xacro:include filename="$(find description)/urdf/imu.xacro" />
-    <xacro:base name="${base_link}" joint_xyz="0 0 ${wheel_radius*2+base_height/2}" />
-    <xacro:lidar name="${lidar_link}" joint_xyz="-${lidar_radius+0.015+0.005} 0 ${lidar_height/2+0.040}" parent_name="${base_link}" />
-    <xacro:camera name="${camera_link}" joint_xyz="${camera_length/2+0.010+0.0675} 0 ${camera_height/2+base_height/2}" parent_name="${base_link}" />
-    <xacro:imu name="${imu_link}" joint_xyz="0 0 ${imu_height/2+base_height/2+0.002}" parent_name="${base_link}" />
-    <xacro:wheel name="${left_front_wheel}" joint_xyz="0.0835 0.0875 -${wheel_radius+base_height/2}" parent_name="${base_link}" />
-    <xacro:wheel name="${left_back_wheel}" joint_xyz="-0.0835 0.0875 -${wheel_radius+base_height/2}" parent_name="${base_link}" />
-    <xacro:wheel name="${right_front_wheel}" joint_xyz="0.0835 -0.0875 -${wheel_radius+base_height/2}" parent_name="${base_link}" />
-    <xacro:wheel name="${right_back_wheel}" joint_xyz="-0.0835 -0.0875 -${wheel_radius+base_height/2}" parent_name="${base_link}" />
+    <xacro:include filename="$(find description)/urdf/chassis.xacro" />
+    <xacro:include filename="$(find description)/urdf/castor.xacro" />
+    <xacro:property name="ground_clearance" value="${castor_radius*2+chassis_height/2}" />
+    <xacro:base name="${base_link}" joint_xyz="0 0 ${wheel_radius}" />
+    <xacro:wheel name="${left_wheel}" joint_xyz="0 ${wheel_width/2} 0" parent_name="${base_link}" />
+    <xacro:wheel name="${right_wheel}" joint_xyz="0 -${wheel_width/2} 0" parent_name="${base_link}" />
+    <xacro:chassis name="${chassis_link}" joint_xyz="${track_width/2} 0 -${wheel_radius-ground_clearance}" parent_name="${base_link}" />
+    <xacro:castor name="${castor_link}" joint_xyz="${track_width/2} 0 -${ground_clearance-castor_radius}" parent_name="${chassis_link}" />
+    <xacro:lidar name="${lidar_link}" joint_xyz="0 0 ${0.106-chassis_height/2}" parent_name="${chassis_link}" />
+    <xacro:imu name="${imu_link}" joint_xyz="0 0 ${0.056-chassis_height/2}" parent_name="${chassis_link}" />
+    <xacro:camera name="${camera_link}" joint_xyz="${track_width/2+0.016} 0 ${0.053+camera_height/2-chassis_height/2}" parent_name="${chassis_link}" />
 </robot>

File: ros2_master/src/description/urdf/base.xacro (robot description, xacro)
@@ -1,28 +1,9 @@
 <?xml version="1.0"?>
 <robot xmlns:xacro="http://ros.org/wiki/xacro" name="base">
-    <xacro:property name="base_length" value="0.210" />
-    <xacro:property name="base_width" value="0.120" />
-    <xacro:property name="base_height" value="0.009" />
     <xacro:property name="link_xyz" value="0 0 0" />
     <xacro:property name="link_rpy" value="0 0 0" />
     <link name="base_footprint" />
     <xacro:macro name="base" params="name joint_xyz">
-        <link name="${name}">
-            <visual>
-                <origin xyz="${link_xyz}" rpy="${link_rpy}" />
-                <geometry>
-                    <box size="${base_length} ${base_height} ${base_width}" />
-                </geometry>
-                <material name="grey">
-                    <color rgba="1 1 1 1" />
-                </material>
-            </visual>
-            <collision>
-                <origin xyz="${link_xyz}" rpy="${link_rpy}" />
-                <geometry>
-                    <box size="${base_length} ${base_height} ${base_width}" />
-                </geometry>
-            </collision>
-        </link>
+        <link name="${name}" />
         <joint name="${name}_joint" type="fixed">
             <origin xyz="${joint_xyz}" rpy="0 0 0" />

File: ros2_master/src/description/urdf/camera.xacro (robot description, xacro)
@@ -1,7 +1,7 @@
 <?xml version="1.0"?>
 <robot xmlns:xacro="http://ros.org/wiki/xacro">
-    <xacro:property name="camera_length" value="0.019" />
-    <xacro:property name="camera_width" value="0.027" />
-    <xacro:property name="camera_height" value="0.042" />
+    <xacro:property name="camera_length" value="0.027" />
+    <xacro:property name="camera_width" value="0.014" />
+    <xacro:property name="camera_height" value="0.040" />
     <xacro:macro name="camera" params="name joint_xyz parent_name">
         <link name="${name}">
@@ -12,5 +12,5 @@
                 </geometry>
                 <material name="orange">
-                    <color rgba="0.0 1.0 1.0 1" />
+                    <color rgba="0.0 1.0 1.0 0.5" />
                 </material>
             </visual>

File: ros2_master/src/description/urdf/imu.xacro (robot description, xacro)
@@ -11,5 +11,5 @@
                 </geometry>
                 <material name="purple">
-                    <color rgba="1.0 0.0 1.0 1" />
+                    <color rgba="1.0 0.0 1.0 0.5" />
                 </material>
             </visual>

File: ros2_master/src/description/urdf/lidar.xacro (robot description, xacro)
@@ -9,6 +9,7 @@
                 <geometry>
                     <cylinder radius="${lidar_radius}" length="${lidar_height}" />
-                </geometry>· <material name="black">
-                    <color rgba="0.0 0.0 1.0 1" />
+                </geometry>
+                <material name="black">
+                    <color rgba="0.0 0.0 1.0 0.5" />
                 </material>
             </visual>

File: ros2_master/src/description/urdf/wheel.xacro (robot description, xacro)
@@ -1,6 +1,6 @@
 <?xml version="1.0"?>
 <robot xmlns:xacro="http://ros.org/wiki/xacro">
-    <xacro:property name="wheel_radius" value="0.0325" />
-    <xacro:property name="wheel_width" value="0.026" />
+    <xacro:property name="wheel_radius" value="0.0335" />
+    <xacro:property name="wheel_height" value="0.026" />
     <xacro:property name="link_xyz" value="0 0 0" />
     <xacro:property name="link_rpy" value="${pi/2} 0 0" />
@@ -10,8 +10,8 @@
                 <origin xyz="${link_xyz}" rpy="${link_rpy}" />
                 <geometry>
-                    <cylinder radius="${wheel_radius}" length="${wheel_width}" />
+                    <cylinder radius="${wheel_radius}" length="${wheel_height}" />
                 </geometry>
                 <material name="yellow">
-                    <color rgba="1.0 1.0 0.0 1" />
+                    <color rgba="1.0 1.0 0.0 0.5" />
                 </material>
             </visual>
@@ -19,5 +19,5 @@
                 <origin xyz="${link_xyz}" rpy="${link_rpy}" />
                 <geometry>
-                    <cylinder radius="${wheel_radius}" length="${wheel_width}" />
+                    <cylinder radius="${wheel_radius}" length="${wheel_height}" />
                 </geometry>
             </collision>
